File: USBPowerBlock/USBPowerBlock.kicad_pcb (KiCad board)
At the start: 2 copper layers, 83.5 x 36.3 mm, 56 parts, among them J1 USB_A, J2 USB_A, J3 USB_A, J4 USB_A, J5 USB_A, J6 IO, J7 Power_In, Q1 LMAK15N10, Q2 LMAK15N10, Q3 LMAK15N10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

Commit message: V2
Fix for V2 stuff up and Assembly Photos
Routing:
- net GND1: track 11.3 -> 21.1 mm
- net GND2: track 11.0 -> 16.2 mm
- net GND5: track 10.6 -> 15.4 mm
- net 5V4: track 6.36 -> 11.2 mm
- net GND4: track 10.8 -> 15.4 mm
- net GND3: track 10.9 -> 15.5 mm
- net 5V5: track 6.46 -> 10.6 mm
- net 5V1: track 6.02 -> 9.15 mm
- net 5V2: track 6.54 -> 9.51 mm
- net 5V3: track 6.53 -> 9.43 mm
- net GND: vias 16 -> 15
Other:
- board text added: "V2"
