File: USBPowerBlock/USBPowerBlock.kicad_sch (KiCad schematic)
At the start: 54 parts, among them J1 USB_A, J2 USB_A, J3 USB_A, J4 USB_A, J5 USB_A, J6 IO, J7 Power_In, Q1 LMAK15N10, Q2 LMAK15N10, Q3 LMAK15N10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

Commit message: V2
Fix for V2 stuff up and Assembly Photos
Parts:
- J1, J2, J3, J4, J5: symbol Connector:USB_A -> USB_A_Socket_Vertical:USB_A_Socket_Vertical
Changed lines of the file:
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@@
 	)
 	(symbol
-		(lib_id "Connector:USB_A")
+		(lib_id "USB_A_Socket_Vertical:USB_A_Socket_Vertical")
 		(at 134.62 48.26 0)
 		(unit 1)
@@
 	)
 	(symbol
-		(lib_id "Connector:USB_A")
+		(lib_id "USB_A_Socket_Vertical:USB_A_Socket_Vertical")
 		(at 198.12 48.26 0)
 		(unit 1)
@@
 	)
 	(symbol
-		(lib_id "Connector:USB_A")
+		(lib_id "USB_A_Socket_Vertical:USB_A_Socket_Vertical")
 		(at 113.03 48.26 0)
 		(unit 1)
@@
 	)
 	(symbol
-		(lib_id "Connector:USB_A")
+		(lib_id "USB_A_Socket_Vertical:USB_A_Socket_Vertical")
 		(at 156.21 48.26 0)
 		(unit 1)
@@
 	)
 	(symbol
-		(lib_id "Connector:USB_A")
+		(lib_id "USB_A_Socket_Vertical:USB_A_Socket_Vertical")
 		(at 176.53 48.26 0)
 		(unit 1)
